File: Hardware/5_phase_C.kicad_sch (KiCad schematic)
At the start: 17 parts

Commit message: feat: Update to use I2C stemma connector
Changed lines of the file:
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@@
 		(company "mangoByte")
+	)
+	(rectangle
+		(start 22.86 36.83)
+		(end 276.86 157.48)
+		(stroke
+			(width 0.2)
+			(type dash)
+		)
+		(fill
+			(type none)
+		)
 	)
 	(text "PA1206FRF470R002L 1W\n@Phase Current=15A, \nV(R_{s})=0.03V, P(R_{s})=0.45W"
